File: power.sch (KiCad schematic (older format))
At the start: 6 parts, among them U1701 tps6240x

Commit message: Layout complete, needs silk screen cleanup and few checks
Signed-off-by: Alexis Jeandet <alexis.jeandet@member.fsf.org>
Parts:
- added C1704, C1705, C1714, C1715, C1716, C1717: 4.7uF, Capacitor_SMD:C_1206_3216Metric_Pad1.42x1.75mm_HandSolder, symbol Device:C
- added C1706: 100nF, Capacitor_SMD:C_0603_1608Metric_Pad1.05x0.95mm_HandSolder, symbol Device:C
- added C1707, C1708, C1709, C1710, C1711, C1723: C, Capacitor_SMD:C_0603_1608Metric_Pad1.05x0.95mm_HandSolder, symbol Device:C
- added C1712, C1713, C1718, C1719, C1721, C1722: 22uF, Capacitor_SMD:C_1206_3216Metric_Pad1.42x1.75mm_HandSolder, symbol Device:C
- added C1720, C1724, C1725: 10uF, Capacitor_SMD:C_1206_3216Metric_Pad1.42x1.75mm_HandSolder, symbol Device:C
- added D1701, D1702: D_Schottky, Diode_SMD:D_SMA_Handsoldering, symbol Device:D_Schottky
- added L1703, L1704, L1705, L1706: 4.7uH, Inductor_SMD:L_1008_2520Metric, symbol Device:L
- added L1707, L1708: 2.2uH, Inductor_SMD:L_1206_3216Metric_Pad1.42x1.75mm_HandSolder, symbol Device:L
- added Q1701: Q_PMOS_GSD, Package_TO_SOT_SMD:SOT-23, symbol Device:Q_PMOS_GSD
- added R1701: 100, Resistor_SMD:R_1206_3216Metric_Pad1.42x1.75mm_HandSolder, symbol Device:R
- added R1702, R1703, R1704, R1705, R1708, R1709, R1710, R1711: R, Resistor_SMD:R_0603_1608Metric_Pad1.05x0.95mm_HandSolder, symbol Device:R
- added R1706, R1707: 500m, Resistor_SMD:R_1206_3216Metric_Pad1.42x1.75mm_HandSolder, symbol Device:R
- added U1702: TPS6513x, Package_DFN_QFN:HVQFN-24-1EP_4x4mm_P0.5mm_EP2.5x2.5mm, symbol TPS6513x:TPS6513x
- added U1703: tps6240x, Package_SON:Texas_S-PVSON-N10_ThermalVias, symbol TPS6240x:tps6240x
Connections:
- net #3.3V: now also C1718.1, L1705.1
- net GND: now also C1704.2, C1705.2, C1706.2, C1707.2, C1708.2, C1710.2, C1712.2, C1713.2, C1714.2, C1715.2, C1716.2, C1717.2, C1718.2, C1719.2, C1720.2, C1721.2, C1722.2, C1724.2, C1725.2, L1704.2, R1705.2, R1709.2, R1711.2, U1702.19 (AGND), U1702.2 (PGND), U1702.25 (PAD), U1702.3 (PGND), U1703.11 (PAD), U1703.2 (MODE/DATA), U1703.8 (GND)
- net USB_5V: now also C1704.1, C1720.1, Q1701.2 (S), R1701.2, U1702.10 (ENN), U1702.11 (PSN), U1702.5 (INN), U1702.6 (INN), U1702.8 (ENP), U1702.9 (PSP), U1703.3 (VIN), U1703.7 (EN_1), U1703.9 (EN_2)
- new net: C1705.1, L1703.1, Q1701.3 (D)
- new net: D1701.2 (A), L1703.2, U1702.1 (INP), U1702.24 (INP)
- new net: Q1701.1 (G), U1702.7 (BSW)
- new net: C1708.1, R1702.1, U1702.17 (VREF)
- new net: C1709.1, R1702.2, R1703.1, U1702.16 (FBN)
- new net: C1706.1, R1701.1, U1702.4 (VIN)
- new net: D1702.1 (K), L1704.1, U1702.13 (OUTN), U1702.14 (OUTN)
- new net: C1707.1, U1702.21 (CP)
- new net: C1710.1, U1702.18 (CN)
- new net: C1711.2, R1704.2, R1705.1, U1702.22 (FBP)
- new net: L1705.2, R1706.2
- new net: L1707.1, U1703.6 (SW1)
- new net: L1708.1, U1703.10 (SW2)
- new net: C1723.2, R1708.2, R1709.1, U1703.1 (ADJ2)
- new net: R1710.2, R1711.1, U1703.5 (DEF1)
- new net: L1706.2, R1707.2
- new net #1.8V: C1725.1, L1707.2, R1710.1, U1703.4 (FB1)
- new net #2.5V: C1721.1, C1723.1, C1724.1, L1706.1, L1708.2, R1708.1
- new net -5V: C1709.2, C1712.1, C1714.1, C1715.1, D1702.2 (A), R1703.2, U1702.15 (VNEG)
- new net 2.5V: C1722.1, R1707.1
- new net 3.3V: C1719.1, R1706.1
- new net 5V: C1711.1, C1713.1, C1716.1, C1717.1, D1701.1 (K), R1704.1, U1702.23 (VPOS)
Other:
- note added: "=======================\n5V -> ADC AOPs ~30mA? + DAC AOP 7mA + ADCs 5mA = 240mA\n=======================\n-5V -> AOPs ~30mA? + DAC AOP 7mA = 210 mA\n=======================\n3.3V -> DACs(60mA) = 120mA max\n=======================\n2.5V -> ADCs(26 mA) = 156mA max\n=======================\n#3.3V -> FPGA(?) + DAC(16mA) = > 150mA?\n=======================\n#2.5V -> FPGA (<10mA) + ADCs(10mA) + LVDS (<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"
- moved on the sheet: C1701, C1702, C1703, L1701, L1702, U1701
