File: SCM_Bench.kicad_pcb (KiCad board)
At the start: 4 copper layers, 86 x 145 mm, 374 parts, among them J101 Conn_Coaxial, J102 Conn_Coaxial, J103 Conn_Coaxial, J104 Conn_Coaxial, J105 Conn_Coaxial, J106 Conn_Coaxial, J107 Conn_02x20_Odd_Even, J108 Conn_02x07_Odd_Even, J109 Conn_02x07_Odd_Even, J110 Conn_Coaxial, J111 Conn_Coaxial, J1601 Conn_01x06, J301 RF_Shield_One_Piece, J401 RF_Shield_One_Piece, J501 RF_Shield_One_Piece, J601 RF_Shield_One_Piece, J701 RF_Shield_One_Piece, J801 RF_Shield_One_Piece, J901 Conn_Coaxial, J902 Conn_Coaxial, J903 Conn_Coaxial, J904 Conn_Coaxial, Q1701 Q_PMOS_GSD, SW1601 SW_Push, U1001 AD9747BCPZ, U1002 SN65LVDS1DBV, U1101 AD8021, U1201 AD8021, U1301 AD9747BCPZ, U1302 SN65LVDS1DBV, U1401 AD8021, U1501 AD8021, U1601 ICE40HX1K-4K-TQ144, U1602 M25PX32-VMW, U1603 ASDMB-xxxMHz, U1701 tps6240x, U1702 TPS6513x, U1703 tps6240x, U301 LT6600IS8, U302 LTC2386-18, U303 SN65LVDS1050PW, U401 LT6600IS8, U402 LTC2386-18, U403 SN65LVDS1050PW, U501 LT6600IS8, U502 LTC2386-18, U503 SN65LVDS1050PW, U601 LT6600IS8, U602 LTC2386-18, U603 SN65LVDS1050PW, U701 LT6600IS8, U702 LTC2386-18, U703 SN65LVDS1050PW, U801 LT6600IS8, U802 LTC2386-18, U803 SN65LVDS1050PW

Commit message: Last cleanups
Signed-off-by: Alexis Jeandet <alexis.jeandet@member.fsf.org>
Parts:
- moved C1703 2.96 mm to (71.1, 158.8), turned to 0 degrees
- moved LOGO102 2.18 mm to (91.4, 41.4)
- moved LOGO101 1.27 mm to (105.2, 42.4)
Routing:
- net GND: vias 479 -> 1159
Other:
- board text added: "CLK"
- board text added: "CS"
- board text added: "GND"
- board text added: "IN 1"
- board text added: "IN 2"
- board text added: "IN 3"
- board text added: "IN 4"
- board text added: "IN 5"
- board text added: "IN 6"
- board text added: "MISO"
- board text added: "MOSI"
- board text added: "OUT 1"
- board text added: "OUT 2"
- board text added: "OUT 3"
- board text added: "OUT 4"
- board text added: "RST"
- board text added: "SCM bench 1.0"
- board text added: "TRIG IN"
- board text added: "TRIG OUT"

Commit message: Desing as ordered for V1.0
Signed-off-by: Alexis Jeandet <alexis.jeandet@member.fsf.org>
Parts:
- U302, U402, U502, U602, U702, U802: footprint Package_DFN_QFN:QFN-32-1EP_5x5mm_P0.5mm_EP3.45x3.45mm_ThermalVias -> Package_DFN_QFN:QFN-32-1EP_5x5mm_P0.5mm_EP3.45x3.45mm
Routing:
- net GND: track 227.2 -> 233.3 mm, vias 1159 -> 1179
